Commit message: added bin 2

File: hrwros_week2/urdf/hrwros_assignment1.xacro (robot description, xacro)
@@ -20,4 +20,5 @@
   <xacro:include filename="$(find hrwros_support)/urdf/bin/bin.urdf.xacro"/>
   <xacro:bin_urdf prefix="bin_1_"/>
+  <xacro:bin_urdf prefix="bin_2_"/>
   <!-- Joints -->
   <joint name="world_interface_to_world" type="fixed">
@@ -63,5 +64,6 @@
     <parent link="world" />
     <child link="robot2_pedestal_link" />
-  </joint>
+  </joint><child link="bin_1_base_link" />
+    <origin xyz="-8.0 -2.2 0" rpy="0 0 0" />
   <xacro:include filename="$(find ur_description)/urdf/ur5.urdf.xacro"/>
   <xacro:ur5_robot prefix="robot2_" joint_limited="true"/>
@@ -71,4 +73,8 @@
     <origin xyz="0 0 0.6" rpy="0 0 ${radians(90)}" />
   </joint>
-  <!-- Add your solution to assignment 1 here -->
+  <joint name="bin_2_joint" type="fixed">
+    <parent link="world_interface" />
+    <child link="bin_2_base_link" />
+    <origin xyz="2.0 1.8 0" rpy="0 0 0" />
+  </joint>
 </robot>
