Commit message: adding gree sphere

File: hrwros_week2/urdf/hrwros_assignment2.xacro (robot description, xacro)
@@ -71,4 +71,19 @@
     <origin xyz="0 0 0.6" rpy="0 0 ${radians(90)}" />
   </joint>
-  <!-- Add your solution to assignment 2 here -->
+<link name="sphere_link">
+    <visual>
+      <origin xyz="0 0 0.0" />
+      <geometry>
+        <sphere radius="0.4" />
+      </geometry>
+      <material name="spehere_link_clr">
+        <color rgba="0 0.9 0 1" />
+      </material>
+    </visual>
+  </link>
+<joint name="sphere_joint" type="fixed">
+  <origin xyz=" 5.8 -5.3 0.4" />
+  <parent link="world"/>
+  <child link="sphere_link"/>
+</joint>
 </robot>
