Commit message: Robot3 added

File: hrwros_week2/urdf/hrwros_assignment3.xacro (robot description, xacro)
@@ -65,10 +65,10 @@
   </joint>
   <!-- Update the below block for assignment 3 here -->
-  <xacro:include filename="$(find ur_description)/urdf/ur5.urdf.xacro"/>
-  <xacro:ur5_robot prefix="robot2_" joint_limited="true"/>
+  <xacro:include filename="$(find hrwros_week2)/urdf/robot/lrmate200ic_macro.xacro"/>
+  <xacro:fanuc_lrmate200ic prefix="robot2_" joint_limited="true"/>
   <joint name="robot2-robot2_pedestal_joint" type="fixed">
     <parent link="robot2_pedestal_link" />
     <child link="robot2_base_link" />
-    <origin xyz="0 0 0.6" rpy="0 0 ${radians(90)}" />
+    <origin xyz="0 0.6 0" rpy="0 0 ${radians(0)}" />
   </joint>
 </robot>
