Commit message: week 3 Assignment

File: hrwros_support/urdf/bin/bin.gazebo.xacro (robot description, xacro)
@@ -12,5 +12,6 @@
     <gazebo>
       <static>true</static>
-      <plugin name="${prefix}object_disposal_plugin" filename="libObjectDisposalPlugin.so">
+<!--
+       <plugin name="${prefix}object_disposal_plugin" filename="libObjectDisposalPlugin.so">
         <contact_sensor_name>${prefix}contact_sensor</contact_sensor_name>
         <contact_side_normal>0 0 1</contact_side_normal>
@@ -18,5 +19,6 @@
         <update_rate>1</update_rate>
       </plugin>
-    </gazebo>
+ -->
+     </gazebo>
   </xacro:macro>
 </robot>

File: hrwros_support/urdf/hrwros.xacro (robot description, xacro)
@@ -17,7 +17,31 @@
   <xacro:include filename="$(find hrwros_support)/urdf/vacuum_gripper/vacuum_gripper.urdf.xacro"/>
   <xacro:vacuum_gripper_urdf prefix="vacuum_gripper1_" joint_prefix="vacuum_gripper1_joint"/>
+  <!-- Robot2 Pedestal -->
+  <xacro:include filename="$(find hrwros_support)/urdf/robot_pedestal/robot_pedestal.urdf.xacro"/>
+  <xacro:robot_pedestal_urdf pedestal_prefix="robot2_" pedestal_parent="world_interface" pedestal_height="0.7">
+    <origin xyz="-7.8 -1.5 0.0" rpy="0 0 0"/>
+  </xacro:robot_pedestal_urdf>
+  <!-- Robot2 -->
+  <xacro:include filename="$(find ur_description)/urdf/ur5.urdf.xacro"/>
+  <xacro:ur5_robot prefix="robot2_" joint_limited="true"/>
+  <!-- Vacuum Gripper2 -->
+  <xacro:include filename="$(find hrwros_support)/urdf/vacuum_gripper/vacuum_gripper.urdf.xacro"/>
+  <xacro:vacuum_gripper_urdf prefix="vacuum_gripper2_" joint_prefix="vacuum_gripper2_joint"/>
   <!-- bins -->
   <xacro:include filename="$(find hrwros_support)/urdf/bin/bin.urdf.xacro"/>
   <xacro:bin_urdf prefix="bin_1_"/>
+  <!-- logical camera 1 collision model -->
+  <xacro:include filename="$(find hrwros_support)/urdf/logical_camera/logical_camera.urdf.xacro"/>
+  <xacro:logical_camera_urdf prefix="logical_camera1_" logical_camera_parent="world_interface">
+    <origin xyz="1.2 1.8 2.0" rpy="0 1.5708 0"/>
+  </xacro:logical_camera_urdf>
+  <!-- logical camera 2 collision model -->
+  <xacro:include filename="$(find hrwros_support)/urdf/logical_camera/logical_camera.urdf.xacro"/>
+  <xacro:logical_camera_urdf prefix="logical_camera2_" logical_camera_parent="world_interface">
+    <origin xyz="-8.3 -1.23 1.8" rpy="0 1.5708 0"/>
+  </xacro:logical_camera_urdf>
+  <!-- break beam -->
+  <xacro:include filename="$(find hrwros_support)/urdf/break_beam/break_beam.urdf.xacro"/>
+  <xacro:break_beam_urdf prefix="break_beam_"/>
   <!-- Joints -->
   <joint name="world_interface_to_world" type="fixed">
@@ -33,6 +57,6 @@
   <!-- robot1 to pedestal. -->
   <joint name="robot1_to_pedestal" type="fixed">
-  <origin xyz="0 0 0.95" rpy="0 0 0" />
-  <parent link="robot1_pedestal_link" />
+  <origin xyz="0.5 1.8 0.95" rpy="0 0 0" />
+  <parent link="world_interface" />
   <child link="robot1_base_link" />
   </joint>
@@ -42,5 +66,27 @@
     <child link="vacuum_gripper1_base_link" />
   </joint>
-  <!-- bin 1 -->
+  <!-- robot2-pedestal to world. -->
+  <joint name="robot2_pedestal_to_world_interface" type="fixed">
+    <parent link="world_interface" />
+    <child link="robot2_pedestal_link" />
+    <origin xyz="-7.8 -1.5 0.0" rpy="0.0 0.0 0.0"/>
+  </joint>
+  <!-- robot2 to pedestal. -->
+  <joint name="robot2_to_pedestal" type="fixed">
+    <parent link="world_interface" />
+    <child link="robot2_base_link" />
+    <origin xyz="-7.8 -1.5 0.7" rpy="0 0 1.57" />
+  </joint>
+  <!-- gripper2 to robot2. -->
+  <joint name="gripper2_to_robot2" type="fixed">
+    <parent link="robot2_tool0" />
+    <child link="vacuum_gripper2_base_link" />
+  </joint>
+  <!-- break beam to world. -->
+  <joint name="break_beam_joint" type="fixed">
+    <parent link="world_interface" />
+    <child link="break_beam_world_interface" />
+  </joint>
+  <!-- bin to world. -->
   <joint name="bin_1_joint" type="fixed">
     <parent link="world_interface" />
@@ -48,26 +94,3 @@
     <origin xyz="-8.0 -2.2 0.0" rpy="0 0 0" />
   </joint>
-  <link name='robot2_pedestal_link'>
-    <visual>
-      <origin xyz="0 0 0.3" />
-      <geometry>
-      <box size="0.3 0.3 0.6" />
-      </geometry>
-      <material name="robot2_pedestal_color">
-        <color rgba=" 0 0.16 0.53 1" />
-      </material>
-    </visual>
-  </link>
-  <joint name="robot2_pedestal_joint" type="fixed">
-    <parent link="world" />
-    <child link="robot2_pedestal_link" />
-    <origin xyz="-7.8 -1.5 0" />
-  </joint>
-  <xacro:include filename="$(find ur_description)/urdf/ur5.urdf.xacro"/>
-  <xacro:ur5_robot prefix="robot2_" joint_limited="true"/>
-  <joint name="robot2-robot_pedestal_joint" type="fixed">
-    <parent link="robot2_pedestal_link"/>
-    <child link="robot2_base_link"/>
-    <origin xyz="0 0 0.6" rpy="0 0 ${radians(90)}"/>
-  </joint>
 </robot>

File: hrwros_support/urdf/vacuum_gripper/vacuum_gripper.gazebo.xacro (robot description, xacro)
@@ -18,5 +18,5 @@
         <suction_cup_link>${gripper_link}</suction_cup_link>
         <!-- ROS -->
-        <robot_namespace>/hrwros</robot_namespace>
+        <!-- <robot_namespace>/hrwros</robot_namespace> -->
         <control_topic>${plugin_name}/control</control_topic>
         <state_topic>${plugin_name}/state</state_topic>

File: hrwros_support/urdf/vacuum_gripper/vacuum_gripper.urdf.xacro (robot description, xacro)
@@ -28,8 +28,32 @@
       </inertial>
     </link>
-    <link name="${prefix}suction_cup"/>
+    <link name="${prefix}suction_cup">
+      <visual>
+        <origin xyz="0 0 0" rpy="0 0 0" />
+        <geometry>
+          <box size="0.001 0.001 0.001" />
+        </geometry>
+        <material name="red">
+          <color rgba="1 0 0 1"/>
+        </material>
+      </visual>
+      <collision>
+        <origin xyz="0 0 0" rpy="0 0 0"/>
+        <geometry>
+          <box size="0.001 0.001 0.001" />
+        </geometry>
+        <material name="red"/>
+      </collision>
+      <inertial>
+        <origin xyz="0 0 0" rpy="0 0 0" />
+        <inertia ixx="0.0001" ixy="0" ixz="0"
+                 iyy="0.0001" iyz="0"
+                 izz="0.0001" />
+        <mass value="0.00001" />
+      </inertial>
+    </link>
     <!-- joint list -->
     <joint name="${joint_prefix}" type="fixed">
-      <origin xyz="0 0 0.080" rpy="0 0 0" />
+      <origin xyz="0 0 0.01" rpy="0 0 0" />
       <parent link="${prefix}base_link" />
       <child link="${prefix}suction_cup" />
